File: TrackingTurrentBoard/GPS.kicad_sch (KiCad schematic)
At the start: 1 part, among them U301 MAX-M8C

Commit message: PCB done
Parts:
- added C301: 100nF, Capacitor_SMD:C_0603_1608Metric, symbol Device:C
- added C302: 1uF, Capacitor_SMD:C_0603_1608Metric, symbol Device:C
- added U302: 734120114, Connector_RF:73412-0114_MOL, symbol Connectors_RF:734120114
Connections:
- net GND: now reaches U301.1 (GND), U301.10 (GND), U301.12 (GND)
- net GND: now also C301.2, C302.2, U302.2 (GROUND), U302.3 (GROUND), U302.4 (GROUND)
- net at U301.11 (RF_IN): now also U302.1 (SIGNAL)
- net SDA: now reaches U301.16 (SDA)
- net SCL: now reaches U301.17 (SCL)
- net GPS_INT: now reaches U301.5 (EXTINT)
- net +3.3V: now reaches U301.7 (VCC_IO)
- net +3.3V: now also U301.8 (VCC), C301.1, C302.1
- net GPS_RST: now reaches U301.9 (~{RESET})
- no-connect marks 0 -> 7
