File: TrackingTurrentBoard/Motors.kicad_sch (KiCad schematic)
At the start: 0 parts

Commit message: PCB done
Parts:
- added C401: 330nF, Capacitor_SMD:C_0603_1608Metric, symbol Device:C
- added C403: 10nF, Capacitor_SMD:C_0603_1608Metric, symbol Device:C
- added C404: 1nF, Capacitor_SMD:C_0603_1608Metric, symbol Device:C
- added C405: 100nF, Capacitor_SMD:C_0603_1608Metric, symbol Device:C
- added C406: 1uF, Capacitor_SMD:C_0603_1608Metric, symbol Device:C
- added J401: Conn_01x02, Connector_PinHeader_2.54mm:PinHeader_1x02_P2.54mm_Vertical, symbol Connector_Generic:Conn_01x02
- added R401, R402: 330m, Resistor_SMD:R_2512_6332Metric, symbol Device:R_US
- added R403: 2.3k, Resistor_SMD:R_0603_1608Metric, symbol Device:R_US
- added R404: 1k, Resistor_SMD:R_0603_1608Metric, symbol Device:R_US
- added R405: 39k, Resistor_SMD:R_0603_1608Metric, symbol Device:R_US
- added R406: 18k, Resistor_SMD:R_0603_1608Metric, symbol Device:R_US
- added R407: 10k, Resistor_SMD:R_0603_1608Metric, symbol Device:R_US
- added U401: STSPIN820, MotorLib:QFN_SPIN820_STM, symbol MotorLib:STSPIN820
Connections:
- new net: C405.1, C406.1, J401.1 (Pin_1), R403.2, R404.1, U401.1 (REF)
- new net: R401.1, U401.4 (SNSA), U401.5 (SENSEA1), U401.6 (SENSEA2)
- new net: R402.1, U401.13 (SENSEB2), U401.14 (SENSEB1), U401.15 (SNSB)
- new net: R407.1, U401.24 (TOFF)
- new net +3.3V: R405.1, R406.1
- new net DECAY: U401.18 (DECAY)
- new net DIR: U401.20 (DIR)
- new net EN\FAULT: C403.1, R405.2, U401.17 (EN\FAULT)
- new net GND: C401.2, C403.2, C404.2, C405.2, C406.2, J401.2 (Pin_2), R401.2, R402.2, R404.2, R407.2, U401.2 (GND), U401.25 (EPAD), U401.3 (GND)
- new net MODE1: U401.21 (MODE1)
- new net MODE2: U401.22 (MODE2)
- new net MODE3: U401.23 (MODE3)
- new net OUTA1: U401.7 (OUTA1)
- new net OUTA2: U401.8 (OUTA2)
- new net OUTB1: U401.11 (OUTB2)
- new net OUTB2: U401.12 (OUTB1)
- new net STBY\RST: C404.1, R406.2, U401.16 (STBY\RESET)
- new net STCK: U401.19 (STCK)
- new net STEP_PWM: R403.1
- new net VBUS: C401.1, U401.10 (VS), U401.9 (VS)
Other:
- note removed: "Need to add footprint and symbol for rotary encoder and motor driver"
