File: TrackingTurrentBoard/Power.kicad_sch (KiCad schematic)
At the start: 14 parts, among them U201 TPS54302, U202 TPS54302

Commit message: added buck sch
Parts:
- removed R201: 511k, Resistor_SMD:R_0603_1608Metric, symbol Device:R_US
- removed R202: 105k, Resistor_SMD:R_0603_1608Metric, symbol Device:R_US
- added C207: 10uF, Capacitor_SMD:C_0603_1608Metric, symbol Device:C
- added C208, C209: 0.1uF, Capacitor_SMD:C_0603_1608Metric, symbol Device:C
- added C210, C211: 22uF, Capacitor_SMD:C_0603_1608Metric, symbol Device:C
- added C212: 45pF, Capacitor_SMD:C_0603_1608Metric, symbol Device:C
- added L201: 6.8uH, symbol Device:L_Iron
- added R208: 50, Resistor_SMD:R_0603_1608Metric, symbol Device:R_US
- added R209: 100k, Resistor_SMD:R_0603_1608Metric, symbol Device:R_US
- added R210: 21.6k, Resistor_SMD:R_0603_1608Metric, symbol Device:R_US
- R203: value 49.9k -> 50
Connections:
- net GND: now also U202.1 (GND), C207.2, C208.2, C210.2, C211.2, R210.2
- net VBUS: now also U202.3 (VIN), C207.1, C208.1
- net +5V: now reaches C204.1, C205.1, L202.2, R203.1
- net at U202.2 (SW): now also C209.2
- net at U202.4 (FB): now also C212.2, R209.2, R210.1
- net at U202.6 (BOOT): now also C209.1, L201.1
- new net: C212.1, R208.2, R209.1
- new net +3.3V: C210.1, C211.1, L201.2, R208.1
Other:
- moved on the sheet: C201, C202, C203, C204, C205, C206, L202, R203, R204, R205, U201

Commit message: PCB done
Parts:
- C212: value 45pF -> 43pF
- L201, L202: footprint (none) -> Inductors:IND_BOURNS_SRP1250
- R210: value 21.6k -> 22.1k
Connections:
- net at C209.1, U202.6 (BOOT): no longer L201.1
- net at C209.2, U202.2 (SW): now also L201.1
- net at C203.2, U201.2 (SW): now also L202.1
- net at C203.1, U201.6 (BOOT): no longer L202.1
Other:
- note added: "3.3V Buck"
- note added: "5V Buck"
- moved on the sheet: C201, C202, C203, C204, C205, C206, C207, C208, C209, C210, C211, C212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
