File: Hardware/TrackingTurrentBoard/TrackingTurrentBoard.kicad_sch (KiCad schematic)
At the start: 37 parts, among them J101 Screw_Terminal_01x04, J102 Conn_01x05, J103 Conn_01x02, J104 Conn_01x03, J105 Conn_01x02, J106 Conn_01x02, J107 Conn_01x02, J108 Screw_Terminal_01x02, J110 2171790001, SW101 SW_MEC_5G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

Commit message: most recent pcb and sch
Parts:
- added C107: 0.1uF, Capacitor_SMD:C_0603_1608Metric, symbol Device:C
- added J109: Conn_01x02, Connector_PinHeader_2.54mm:PinHeader_1x02_P2.54mm_Vertical, symbol Connector_Generic:Conn_01x02
- added SW102: SW_MEC_5G, Button_Switch_SMD:SW_SPST_CK_RS282G05A3, symbol Switch:SW_MEC_5G
Connections:
- net FTDI_RX: now also U101.21 (PB10); no longer U101.22 (PB11)
- net FTDI_TX: now also U101.22 (PB11); no longer U101.21 (PB10)
- net GND: now also C107.2, SW102.1 (A)
- net RESET: now reaches C101.1, SW101.2 (B), U101.7 (NRST)
- net SWCLK: now reaches U101.34 (PA13)
- net SWCLK: now also J109.1 (Pin_1)
- net SWDIO: now reaches U101.37 (PA14)
- net SWDIO: now also J109.2 (Pin_2)
- net BOOT: now reaches U101.44 (PH3)
- net BOOT: now also C107.1, SW102.2 (B)
- no-connect marks 30 -> 27
Other:
- moved on the sheet: C101, SW101
